File: Schematics/Preliminary/Pre_sch.brd (EAGLE design)
At the start: 100 x 40 mm, 39 parts, among them IC1 7805TV, IC2 7805TV, J1 3x2 M, J2 1x6 M, SW1 !RESET, SW2 Unlock, U2 A4988_STEPPER_MOTOR_DRIVER_CA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, U4 ATMEGA328P-PU, X1 16 MHz

Commit message: Better board template; still needs rearranging
Parts:
- moved R7 287.3 mm to (-36.8, 147.3)
- moved SW2 281.9 mm to (-100.3, 147.3)
- moved H4 233.3 mm to (-86.4, 147.3)
- moved C1 229.2 mm to (-34.3, 154.9)
- moved J2 228.3 mm to (-100.3, 137.2), turned to 0 degrees
- moved U$2 223.4 mm to (-74.9, 118.1)
- moved C10 222.6 mm to (-16.5, 154.9)
- moved C11 218.2 mm to (-21.6, 154.9)
- moved C5 214.4 mm to (-111.8, 147.3)
- moved C4 214.0 mm to (-106.7, 147.3), turned to 0 degrees
- moved C12 213.9 mm to (-26.7, 154.9)
- moved C6 213.8 mm to (-116.8, 147.3)
- moved TP6 210.2 mm to (-62.2, 153.7)
- moved C13 209.6 mm to (-30.5, 154.9)
- moved SW1 208.1 mm to (-92.7, 147.3)
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Routing:
- net +5V: track 93.5 -> 0.00 mm
- net MOSI: track 61.0 -> 0.00 mm
- net SCK: track 58.9 -> 0.00 mm
- net MISO: track 54.3 -> 0.00 mm
- net !RESET: track 39.6 -> 0.00 mm
- net AVR-TXD: track 23.6 -> 0.00 mm
- net AVR-RXD: track 19.9 -> 0.00 mm
- net XTAL2: track 14.5 -> 0.00 mm
- net XTAL1: track 14.4 -> 0.00 mm
- net N$5: track 3.87 -> 0.00 mm
- net FTDI-RXD: track 3.51 -> 0.00 mm
- net FTDI-TXD: track 3.50 -> 0.00 mm
- net N$1: track 3.20 -> 0.00 mm
- net N$3: track 2.10 -> 0.00 mm
- removed copper zone on layer 1, net GND
- removed copper zone on layer 16, net GND
Other:
- board size 100 x 40 mm -> 160 x 100 mm
- board text removed: "1-BLK"
- board text removed: "D:/SmartProjects/Snc/a4_bn_logo2.bmp"
- board text removed: "ECE411 328 Board Rev 1 Based on Arduino UNO Rev 3 CC by-SA"
- board text removed: "ISP"
- board text removed: "RXD"
- board text removed: "TXD"
- board text removed: "UART"

Commit message: Preliminary Board Layout is done
Parts:
- C1: value 48u -> 100u
- moved SW2 230.1 mm to (102.9, 39.4), turned to 270 degrees
- moved H4 224.1 mm to (104.1, 29.2)
- moved U$3 218.1 mm to (119.4, 101.6), turned to 270 degrees
- moved SW1 205.6 mm to (102.9, 83.8)
- moved H3 191.7 mm to (104.1, 94.0)
- moved C8 176.0 mm to (80.0, 27.9), turned to 180 degrees
- moved C7 170.9 mm to (76.2, 27.9)
- moved R7 169.6 mm to (94.0, 39.4)
- moved J1 168.8 mm to (95.2, 68.6), turned to 90 degrees
- moved TP3 165.9 mm to (100.3, 77.5)
- moved H2 163.1 mm to (3.81, 3.81)
- moved C1 152.4 mm to (63.5, 38.1)
- moved C4 150.5 mm to (26.7, 77.5)
- moved C6 149.7 mm to (8.89, 66.0)
- moved U$2 149.5 mm to (71.1, 86.4), turned to 270 degrees
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Routing:
- net GND: track 0.00 -> 349.3 mm, vias 0 -> 1
- net +5V: track 0.00 -> 308.8 mm, vias 0 -> 1
- net +12V: track 0.00 -> 147.0 mm
- net N$1: track 0.00 -> 72.6 mm, vias 0 -> 1
- net AVR-RXD: track 0.00 -> 68.7 mm
- net !RESET: track 0.00 -> 55.3 mm
- net N$6: track 0.00 -> 49.8 mm
- net N$12: track 0.00 -> 49.8 mm
- net AVR-TXD: track 0.00 -> 48.2 mm
- net N$4: track 0.00 -> 39.7 mm
- net N$2: track 0.00 -> 39.7 mm
- net N$20: track 0.00 -> 39.0 mm
- net SCK: track 0.00 -> 37.8 mm
- net MOSI: track 0.00 -> 37.4 mm
- net N$8: track 0.00 -> 37.1 mm
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Other:
- board size 160 x 100 mm -> 120.7 x 109.2 mm
