File: Schematics/Final/schV2.2.brd (EAGLE design)
At the start: 95.4 x 58.6 mm, 41 parts, among them J1 3x2 M, J2 1x6 M, J4 POWER_JACK, SW1 !RESET, SW2 Unlock, U4 ATMEGA328P-PU, X1 16 MHz

Commit message: Add files via upload
Parts:
- removed U$3: pad, keypad_4x4_raw:KEYPAD4X4
- added JP8, JP9: (no value), pinhead:1X04
- moved H2 3.88 mm to (22.9, 86.3)
Connections:
- net MISO: now also JP8.2; no longer U$3.2
- net MOSI: now also JP8.3; no longer U$3.3
- net N$14: now also JP9.1; no longer U$3.8
- net N$15: now also JP9.2; no longer U$3.7
- net N$16: now also JP9.3; no longer U$3.6
- net N$17: now also JP9.4; no longer U$3.5
- net N$18: now also JP8.4; no longer U$3.4
- net SCK: now also JP8.1; no longer U$3.1
Routing:
- net N$17: track 0.00 -> 27.4 mm, vias 0 -> 1
- net N$14: track 69.0 -> 67.7 mm
- net MISO: track 28.3 -> 29.5 mm
- net N$18: track 28.2 -> 29.4 mm
- net SCK: track 42.1 -> 42.8 mm
Other:
- board size 95.4 x 58.6 mm -> 95.4 x 60.4 mm
- board text added: "ece-411-t05-doorlock Cam Osborn Daniel Sayenko Thomas Courcy Abdullah Almarzouq"
