File: Schematics/Final/schV2.2.sch (EAGLE design)
At the start: 41 parts, among them J1 3x2 M, J2 1x6 M, J4 POWER_JACK, SW1 !RESET, SW2 Unlock, U4 ATMEGA328P-PU, X1 16 MHz

Commit message: Add files via upload
Parts:
- removed U$3: pad, keypad_4x4_raw:KEYPAD4X4
- added JP8, JP9: (no value), pinhead:PINHD-1X4
Connections:
- net MISO: now also JP8.2; no longer U$3.C2
- net MOSI: now also JP8.3; no longer U$3.C3
- net N$14: now also JP9.1; no longer U$3.R4
- net N$15: now also JP9.2; no longer U$3.R3
- net N$16: now also JP9.3; no longer U$3.R2
- net N$17: now also JP9.4; no longer U$3.R1
- net N$18: now also JP8.4; no longer U$3.C4
- net SCK: now also JP8.1; no longer U$3.C1
Changed lines of the file:
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@@
 <part name="GND9" library="supply1" library_urn="urn:adsk.eagle:library:371" deviceset="GND" device=""/>
 <part name="P+10" library="supply1" library_urn="urn:adsk.eagle:library:371" deviceset="+5V" device=""/>
-<part name="U$3" library="keypad_4x4_raw" deviceset="KEYPAD4X4" device="" value="pad"/>
 <part name="P+11" library="supply1" deviceset="+5V" device=""/>
 <part name="GND10" library="supply1" deviceset="GND" device=""/>
@@
 <part name="JP6" library="pinhead" library_urn="urn:adsk.eagle:library:325" deviceset="PINHD-1X3" device="" package3d_urn="urn:adsk.eagle:package:22458/2" value="VCC.1 | IN1 | GND"/>
 <part name="JP7" library="pinhead" library_urn="urn:adsk.eagle:library:325" deviceset="PINHD-1X2" device="" package3d_urn="urn:adsk.eagle:package:22435/2" value="COM | NO"/>
+<part name="JP8" library="pinhead" library_urn="urn:adsk.eagle:library:325" deviceset="PINHD-1X4" device="" package3d_urn="urn:adsk.eagle:package:22407/2"/>
+<part name="JP9" library="pinhead" library_urn="urn:adsk.eagle:library:325" deviceset="PINHD-1X4" device="" package3d_urn="urn:adsk.eagle:package:22407/2"/>
 </parts>
 <sheets>
@@
 <attribute name="VALUE" x="325.12" y="101.6" size="1.778" layer="96" rot="R180"/>
 </instance>
-<instance part="U$3" gate="G$1" x="78.74" y="68.58" smashed="yes">
-<attribute name="NAME" x="60.96" y="83.82" size="1.27" layer="95"/>
-<attribute name="VALUE" x="68.58" y="83.82" size="1.27" layer="96"/>
-</instance>
 <instance part="P+11" gate="1" x="106.68" y="207.01" smashed="yes">
 <attribute name="VALUE" x="108.585" y="209.55" size="1.778" layer="96" rot="R180"/>
@@
 <attribute name="NAME" x="120.015" y="229.87" size="1.778" layer="95" rot="R270"/>
 <attribute name="VALUE" x="109.22" y="219.71" size="1.778" layer="96"/>
+</instance>
+<instance part="JP8" gate="A" x="68.58" y="63.5" smashed="yes" rot="R90">
+<attribute name="NAME" x="60.325" y="57.15" size="1.778" layer="95" rot="R90"/>
+<attribute name="VALUE" x="76.2" y="57.15" size="1.778" layer="96" rot="R90"/>
+</instance>
+<instance part="JP9" gate="A" x="78.74" y="76.2" smashed="yes" rot="R180">
+<attribute name="NAME" x="85.09" y="67.945" size="1.778" layer="95" rot="R180"/>
+<attribute name="VALUE" x="85.09" y="83.82" size="1.778" layer="96" rot="R180"/>
 </instance>
 </instances>
@@
 <pinref part="J1" gate="A" pin="3"/>
 <pinref part="U4" gate="G$1" pin="(SCK)PB5"/>
-<pinref part="U$3" gate="G$1" pin="C1"/>
 <wire x1="63.5" y1="60.96" x2="63.5" y2="53.34" width="0.1524" layer="91"/>
 <wire x1="63.5" y1="53.34" x2="142.24" y2="53.34" width="0.1524" layer="91"/>
@@
 <wire x1="142.24" y1="146.05" x2="137.16" y2="146.05" width="0.1524" layer="91"/>
 <junction x="137.16" y="146.05"/>
+<pinref part="JP8" gate="A" pin="1"/>
 </segment>
 </net>
@@
 <pinref part="J1" gate="A" pin="1"/>
 <pinref part="U4" gate="G$1" pin="(MISO)PB4"/>
-<pinref part="U$3" gate="G$1" pin="C2"/>
 <wire x1="66.04" y1="60.96" x2="66.04" y2="55.88" width="0.1524" layer="91"/>
 <wire x1="66.04" y1="55.88" x2="144.78" y2="55.88" width="0.1524" layer="91"/>
@@
 <wire x1="144.78" y1="143.51" x2="137.16" y2="143.51" width="0.1524" layer="91"/>
 <junction x="137.16" y="143.51"/>
+<pinref part="JP8" gate="A" pin="2"/>
 </segment>
 </net>
@@
 <pinref part="J1" gate="A" pin="4"/>
 <pinref part="U4" gate="G$1" pin="(MOSI)PB3"/>
-<pinref part="U$3" gate="G$1" pin="C3"/>
 <wire x1="68.58" y1="60.96" x2="68.58" y2="58.42" width="0.1524" layer="91"/>
 <wire x1="68.58" y1="58.42" x2="147.32" y2="58.42" width="0.1524" layer="91"/>
@@
 <wire x1="147.32" y1="140.97" x2="137.16" y2="140.97" width="0.1524" layer="91"/>
 <junction x="137.16" y="140.97"/>
+<pinref part="JP8" gate="A" pin="3"/>
 </segment>
 </net>
@@
 <net name="N$14" class="0">
 <segment>
-<pinref part="U$3" gate="G$1" pin="R4"/>
 <wire x1="81.28" y1="71.12" x2="157.48" y2="71.12" width="0.1524" layer="91"/>
 <wire x1="157.48" y1="71.12" x2="157.48" y2="107.95" width="0.1524" layer="91"/>
 <pinref part="U4" gate="G$1" pin="(AIN0)PD6"/>
 <wire x1="157.48" y1="107.95" x2="137.16" y2="107.95" width="0.1524" layer="91"/>
+<pinref part="JP9" gate="A" pin="1"/>
 </segment>
 </net>
 <net name="N$15" class="0">
 <segment>
-<pinref part="U$3" gate="G$1" pin="R3"/>
 <wire x1="81.28" y1="73.66" x2="160.02" y2="73.66" width="0.1524" layer="91"/>
 <pinref part="U4" gate="G$1" pin="(AIN1)PD7"/>
 <wire x1="160.02" y1="73.66" x2="160.02" y2="110.49" width="0.1524" layer="91"/>
 <wire x1="160.02" y1="110.49" x2="137.16" y2="110.49" width="0.1524" layer="91"/>
+<pinref part="JP9" gate="A" pin="2"/>
 </segment>
 </net>
 <net name="N$16" class="0">
 <segment>
-<pinref part="U$3" gate="G$1" pin="R2"/>
 <wire x1="81.28" y1="76.2" x2="154.94" y2="76.2" width="0.1524" layer="91"/>
 <wire x1="154.94" y1="76.2" x2="154.94" y2="133.35" width="0.1524" layer="91"/>
 <pinref part="U4" gate="G$1" pin="(ICP)PB0"/>
 <wire x1="154.94" y1="133.35" x2="137.16" y2="133.35" width="0.1524" layer="91"/>
+<pinref part="JP9" gate="A" pin="3"/>
 </segment>
 </net>
 <net name="N$17" class="0">
 <segment>
-<pinref part="U$3" gate="G$1" pin="R1"/>
 <wire x1="81.28" y1="78.74" x2="152.4" y2="78.74" width="0.1524" layer="91"/>
 <wire x1="152.4" y1="78.74" x2="152.4" y2="135.89" width="0.1524" layer="91"/>
 <pinref part="U4" gate="G$1" pin="(OC1)PB1"/>
 <wire x1="152.4" y1="135.89" x2="137.16" y2="135.89" width="0.1524" layer="91"/>
+<pinref part="JP9" gate="A" pin="4"/>
 </segment>
 </net>
 <net name="N$18" class="0">
 <segment>
-<pinref part="U$3" gate="G$1" pin="C4"/>
 <wire x1="71.12" y1="60.96" x2="149.86" y2="60.96" width="0.1524" layer="91"/>
 <wire x1="149.86" y1="60.96" x2="149.86" y2="138.43" width="0.1524" layer="91"/>
 <pinref part="U4" gate="G$1" pin="(SS)PB2"/>
 <wire x1="149.86" y1="138.43" x2="137.16" y2="138.43" width="0.1524" layer="91"/>
-</segment>
-</net>
+<pinref part="JP8" gate="A" pin="4"/>
+</segment>
+</net>
